File: power_supply.kicad_sch (KiCad schematic)
At the start: 10 parts, among them U3 TPS562201

Commit message: Board v2 - reduced size
Parts:
- L1: footprint Inductor_SMD:L_Wuerth_HCI-7030 -> tme_library:VLS6045AF
- R13, R14: footprint Resistor_SMD:R_0402_1005Metric -> Resistor_SMD:R_0402_1005Metric_Pad0.72x0.64mm_HandSolder
Changed lines of the file:
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@@
     (property "Reference" "L1" (id 0) (at 163.322 91.44 90))
     (property "Value" "3u3" (id 1) (at 163.322 93.98 90))
-    (property "Footprint" "Inductor_SMD:L_Wuerth_HCI-7030" (id 2) (at 163.322 97.79 0)
+    (property "Footprint" "tme_library:VLS6045AF" (id 2) (at 163.322 97.79 0)
       (effects (font (size 1.27 1.27)) hide)
     )
@@
       (effects (font (size 1.27 1.27)) (justify left))
     )
-    (property "Footprint" "Resistor_SMD:R_0402_1005Metric" (id 2) (at 168.529 101.6 90)
+    (property "Footprint" "Resistor_SMD:R_0402_1005Metric_Pad0.72x0.64mm_HandSolder" (id 2) (at 168.529 101.6 90)
       (effects (font (size 1.27 1.27)) hide)
     )
@@
       (effects (font (size 1.27 1.27)) (justify left))
     )
-    (property "Footprint" "Resistor_SMD:R_0402_1005Metric" (id 2) (at 168.529 111.76 90)
+    (property "Footprint" "Resistor_SMD:R_0402_1005Metric_Pad0.72x0.64mm_HandSolder" (id 2) (at 168.529 111.76 90)
       (effects (font (size 1.27 1.27)) hide)
     )
