File: _autosave-stm_v3.kicad_sch (KiCad schematic)
At the start: 38 parts, among them Q1 s8050, Q2 s8050, SW1 RST, SW2 BOOT0, U1 STM32L431RCTx, U2 SN65HVD231, Y1 16 MHz

Commit message: Final board version
Parts:
- removed H1: MountingHole, MountingHole:MountingHole_2.7mm_M2.5, symbol Mechanical:MountingHole
Changed lines of the file:
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@@
     (pin "4")
-  )
-  (symbol (lib_id "Mechanical:MountingHole") (at 145.542 160.02 0) (unit 1)
-    (in_bom yes) (on_board yes) (fields_autoplaced)
-    (property "Reference" "H1" (id 0) (at 148.59 158.7499 0)
-      (effects (font (size 1.27 1.27)) (justify left))
-    )
-    (property "Value" "MountingHole" (id 1) (at 148.59 161.2899 0)
-      (effects (font (size 1.27 1.27)) (justify left))
-    )
-    (property "Footprint" "MountingHole:MountingHole_2.7mm_M2.5" (id 2) (at 145.542 160.02 0)
-      (effects (font (size 1.27 1.27)) hide)
-    )
-    (property "Datasheet" "~" (id 3) (at 145.542 160.02 0)
-      (effects (font (size 1.27 1.27)) hide)
-    )
   )
   (symbol (lib_id "power:GND") (at 79.502 170.18 0) (unit 1)
@@
       (reference "D2") (unit 1) (value "LED") (footprint "LED_SMD:LED_0603_1608Metric")
     )
-    (path "/63fbc116-50cb-406d-ba91-edb36459c467"
-      (reference "H1") (unit 1) (value "MountingHole") (footprint "MountingHole:MountingHole_2.7mm_M2.5")
-    )
     (path "/d1937b74-21dd-49cd-bda0-e1e72be87ee5/19750a19-9304-4b77-900a-3960d1ce3fce"
