File: KiCAD project/Diagnostic tool v2/diagnostic_tool_v2/diagnostic_tool_v2.kicad_sch (KiCad schematic)
At the start: 42 parts, among them J1 OBDII, J2 OLED, J3 SWD, Q1 NPN, Q2 NPN, SW1 NRST, SW2 MENU, U1 STM32L431RCTx, U2 SN65HVD231, U3 SN78MCDCYR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

Commit message: Update 26/06/23 - Thesis release
Parts:
- removed SW1: NRST, tme_library:XKB_TS_1187A, symbol Switch:SW_Push
Other:
- moved on the sheet: C10
Changed lines of the file:
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@@
   (junction (at 63.754 73.66) (diameter 0) (color 0 0 0 0)
   )
-  (junction (at 42.926 88.9) (diameter 0) (color 0 0 0 0)
-  )
   (junction (at 48.26 32.766) (diameter 0) (color 0 0 0 0)
   )
@@
   )
   (junction (at 92.456 182.118) (diameter 0) (color 0 0 0 0)
-  )
-  (junction (at 31.75 95.25) (diameter 0) (color 0 0 0 0)
   )
   (junction (at 245.364 41.656) (diameter 0) (color 0 0 0 0)
@@
     (stroke (width 0) (type default))
   )
-  (wire (pts (xy 31.75 95.25) (xy 31.75 101.6))
+  (wire (pts (xy 31.75 88.9) (xy 31.75 101.6))
     (stroke (width 0) (type default))
   )
@@
     (stroke (width 0) (type default))
   )
-  (wire (pts (xy 40.64 95.25) (xy 42.926 95.25))
+  (wire (pts (xy 40.64 88.9) (xy 47.244 88.9))
     (stroke (width 0) (type default))
   )
@@
     (stroke (width 0) (type default))
   )
-  (wire (pts (xy 31.75 88.9) (xy 31.75 95.25))
-    (stroke (width 0) (type default))
-  )
-  (wire (pts (xy 42.926 88.9) (xy 47.244 88.9))
-    (stroke (width 0) (type default))
-  )
   (wire (pts (xy 213.106 88.9) (xy 209.296 88.9))
     (stroke (width 0) (type default))
@@
     (stroke (width 0) (type default))
   )
-  (wire (pts (xy 41.91 88.9) (xy 42.926 88.9))
-    (stroke (width 0) (type default))
-  )
   (wire (pts (xy 231.14 149.352) (xy 231.14 153.162))
     (stroke (width 0) (type default))
@@
     (stroke (width 0) (type default))
   )
-  (wire (pts (xy 31.75 95.25) (xy 33.02 95.25))
+  (wire (pts (xy 31.75 88.9) (xy 33.02 88.9))
     (stroke (width 0) (type default))
   )
@@
   )
   (wire (pts (xy 77.216 101.854) (xy 77.216 103.886))
-    (stroke (width 0) (type default))
-  )
-  (wire (pts (xy 42.926 95.25) (xy 42.926 88.9))
     (stroke (width 0) (type default))
   )
@@
     )
   )
-  (symbol (lib_id "Device:C") (at 36.83 95.25 90) (mirror x) (unit 1)
+  (symbol (lib_id "Device:C") (at 36.83 88.9 90) (mirror x) (unit 1)
     (in_bom yes) (on_board yes) (dnp no)
-    (property "Reference" "C10" (at 36.83 91.948 90)
-      (effects (font (size 1.27 1.27)))
-    )
-    (property "Value" "100n" (at 36.83 99.06 90)
-      (effects (font (size 1.27 1.27)))
-    )
-    (property "Footprint" "Capacitor_SMD:C_0402_1005Metric" (at 40.64 96.2152 0)
-      (effects (font (size 1.27 1.27)) hide)
-    )
-    (property "Datasheet" "~" (at 36.83 95.25 0)
+    (property "Reference" "C10" (at 36.83 85.598 90)
+      (effects (font (size 1.27 1.27)))
+    )
+    (property "Value" "100n" (at 36.83 92.71 90)
+      (effects (font (size 1.27 1.27)))
+    )
+    (property "Footprint" "Capacitor_SMD:C_0402_1005Metric" (at 40.64 89.8652 0)
+      (effects (font (size 1.27 1.27)) hide)
+    )
+    (property "Datasheet" "~" (at 36.83 88.9 0)
       (effects (font (size 1.27 1.27)) hide)
     )
@@
         )
       )
-    )
-  )
-  (symbol (lib_id "Switch:SW_Push") (at 36.83 88.9 0) (unit 1)
-    (in_bom yes) (on_board yes) (dnp no) (fields_autoplaced)
-    (property "Reference" "SW1" (at 36.83 81.788 0)
-      (effects (font (size 1.27 1.27)))
-    )
-    (property "Value" "NRST" (at 36.83 84.328 0)
-      (effects (font (size 1.27 1.27)))
-    )
-    (property "Footprint" "tme_library:XKB_TS_1187A" (at 36.83 83.82 0)
-      (effects (font (size 1.27 1.27)) hide)
-    )
-    (property "Datasheet" "~" (at 36.83 83.82 0)
-      (effects (font (size 1.27 1.27)) hide)
-    )
-    (pin "1")
-    (pin "2")
-    (instances
-      (project "diagnostic_tool_v2"
-        (path "/0d3336a9-dfd3-40fe-814c-79a1ffc561aa"
-          (reference "SW1") (unit 1)
-        )
-      )
