File: KiCAD project/Diagnostic tool with IoT/iot_diagnostic_tool/car.kicad_sch (KiCad schematic)
At the start: 17 parts, among them Q1 s8050, Q2 s8050, U3 SN65HVD231

Commit message: Update 03/03/23 - new schematic done
Connections:
- net +3.3V renamed +3V3
Other:
- note added: "Car communication circuitry"
- moved on the sheet: C18, C19, C20, D1, Q1, Q2, R10, R11, R12, R13, R4, R5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

Commit message: Update 06/03/23 - new board layout WIP 70%
Parts:
- C18: footprint (none) -> Capacitor_SMD:C_0402_1005Metric
- C19, C20: footprint (none) -> Capacitor_SMD:C_0402_1005Metric_Pad0.74x0.62mm_HandSolder
- D1: footprint Package_TO_SOT_SMD_AKL:SOT-23 -> Package_TO_SOT_SMD:SOT-23
- Q1, Q2: footprint (none) -> Package_TO_SOT_SMD:SOT-23
- R10, R11, R12, R13, R4, R5, R6, R7, R8, R9: footprint (none) -> Resistor_SMD:R_0402_1005Metric
Changed lines of the file:
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@@
       (effects (font (size 1.27 1.27)) (justify left))
     )
-    (property "Footprint" "" (at 88.392 146.685 90)
+    (property "Footprint" "Resistor_SMD:R_0402_1005Metric" (at 88.392 146.685 90)
       (effects (font (size 1.27 1.27)) hide)
     )
@@
       (effects (font (size 1.27 1.27)) (justify right))
     )
-    (property "Footprint" "Package_TO_SOT_SMD_AKL:SOT-23" (at 110.49 85.09 0)
+    (property "Footprint" "Package_TO_SOT_SMD:SOT-23" (at 110.49 85.09 0)
       (effects (font (size 1.27 1.27)) hide)
     )
@@
       (effects (font (size 1.27 1.27)) (justify left))
     )
-    (property "Footprint" "" (at 188.722 94.615 90)
+    (property "Footprint" "Resistor_SMD:R_0402_1005Metric" (at 188.722 94.615 90)
       (effects (font (size 1.27 1.27)) hide)
     )
@@
       (effects (font (size 1.27 1.27)) (justify left))
     )
-    (property "Footprint" "" (at 90.5002 95.25 0)
+    (property "Footprint" "Capacitor_SMD:C_0402_1005Metric_Pad0.74x0.62mm_HandSolder" (at 90.5002 95.25 0)
       (effects (font (size 1.27 1.27)) hide)
     )
@@
       (effects (font (size 1.27 1.27)) (justify left))
     )
-    (property "Footprint" "" (at 188.722 83.82 90)
+    (property "Footprint" "Resistor_SMD:R_0402_1005Metric" (at 188.722 83.82 90)
       (effects (font (size 1.27 1.27)) hide)
     )
@@
       (effects (font (size 1.27 1.27)))
     )
-    (property "Footprint" "" (at 168.91 75.057 90)
+    (property "Footprint" "Resistor_SMD:R_0402_1005Metric" (at 168.91 75.057 90)
       (effects (font (size 1.27 1.27)) hide)
     )
@@
       (effects (font (size 1.27 1.27)) (justify left))
     )
-    (property "Footprint" "" (at 88.392 135.89 90)
+    (property "Footprint" "Resistor_SMD:R_0402_1005Metric" (at 88.392 135.89 90)
       (effects (font (size 1.27 1.27)) hide)
     )
@@
       (effects (font (size 1.27 1.27)) (justify left))
     )
-    (property "Footprint" "" (at 234.442 66.04 90)
+    (property "Footprint" "Resistor_SMD:R_0402_1005Metric" (at 234.442 66.04 90)
       (effects (font (size 1.27 1.27)) hide)
     )
@@
       (effects (font (size 1.27 1.27)) (justify left))
     )
-    (property "Footprint" "" (at 241.3 76.835 0)
+    (property "Footprint" "Package_TO_SOT_SMD:SOT-23" (at 241.3 76.835 0)
       (effects (font (size 1.27 1.27)) hide)
     )
@@
       (effects (font (size 1.27 1.27)))
     )
-    (property "Footprint" "" (at 224.79 75.692 90)
+    (property "Footprint" "Resistor_SMD:R_0402_1005Metric" (at 224.79 75.692 90)
       (effects (font (size 1.27 1.27)) hide)
     )
@@
       (effects (font (size 1.27 1.27)) (justify left))
     )
-    (property "Footprint" "" (at 297.18 77.47 0)
+    (property "Footprint" "Package_TO_SOT_SMD:SOT-23" (at 297.18 77.47 0)
       (effects (font (size 1.27 1.27)) hide)
     )
@@
       (effects (font (size 1.27 1.27)) (justify left))
     )
-    (property "Footprint" "" (at 87.757 81.28 90)
+    (property "Footprint" "Resistor_SMD:R_0402_1005Metric" (at 87.757 81.28 90)
       (effects (font (size 1.27 1.27)) hide)
     )
@@
       (effects (font (size 1.27 1.27)) (justify left))
     )
-    (property "Footprint" "" (at 100.457 81.28 90)
+    (property "Footprint" "Resistor_SMD:R_0402_1005Metric" (at 100.457 81.28 90)
       (effects (font (size 1.27 1.27)) hide)
     )
@@
       (effects (font (size 1.27 1.27)) (justify left))
     )
-    (property "Footprint" "" (at 178.562 65.405 90)
+    (property "Footprint" "Resistor_SMD:R_0402_1005Metric" (at 178.562 65.405 90)
       (effects (font (size 1.27 1.27)) hide)
     )
@@
       (effects (font (size 1.27 1.27)) (justify left))
     )
-    (property "Footprint" "" (at 44.1452 77.47 0)
+    (property "Footprint" "Capacitor_SMD:C_0402_1005Metric" (at 44.1452 77.47 0)
       (effects (font (size 1.27 1.27)) hide)
     )
@@
       (effects (font (size 1.27 1.27)) (justify left))
     )
-    (property "Footprint" "" (at 103.2002 95.25 0)
-      (effects (font (size 1.27 1.27)) hide)
-    )
+    (property "Footprint" "Capacitor_SMD:C_0402_1005Metric_Pad0.74x0.62mm_HandSolder" (at 103.2002 95.25 0)
+      (effects (font (size 1.27 1.27)) hide)
+    )

Commit message: Update 17/03/23 - final board update, generated files for manufacturing
Parts:
- removed Q1, Q2: s8050, Package_TO_SOT_SMD:SOT-23, symbol Simulation_SPICE:NPN
- added Q1, Q4: BC817, Package_TO_SOT_SMD:SOT-23, symbol PCM_Transistor_BJT_AKL:BC817
Connections:
- net GND: now also Q1.2 (E), Q4.2 (E)
- net ISO_K: now also Q1.3 (C)
- net ISO_L: now also Q4.3 (C)
- net at R6.1: now also Q1.1 (B)
- net at R8.1: now also Q4.1 (B)
Changed lines of the file:
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@@
+    )
+  )
+  (symbol (lib_id "PCM_Transistor_BJT_AKL:BC817") (at 233.68 77.47 0) (unit 1)
+    (in_bom yes) (on_board yes) (dnp no) (fields_autoplaced)
+    (property "Reference" "Q4" (at 239.395 76.835 0)
+      (effects (font (size 1.27 1.27)) (justify left))
+    )
+    (property "Value" "BC817" (at 239.395 79.375 0)
+      (effects (font (size 1.27 1.27)) (justify left))
+    )
+    (property "Footprint" "Package_TO_SOT_SMD:SOT-23" (at 238.76 74.93 0)
+      (effects (font (size 1.27 1.27)) hide)
+    )
+    (property "Datasheet" "https://www.tme.eu/Document/7b5ea7386544f524d0315334956093bb/BC817-16.215.pdf" (at 233.68 77.47 0)
+      (effects (font (size 1.27 1.27)) hide)
+    )
+    (pin "1")
+    (pin "2")
+    (pin "3")
+    (instances
+      (project "iot_diagnostic_tool"
+        (path "/2db85604-c96b-49da-91cc-aa2116c9cadf/7d43596b-0e17-496e-8cfa-ffe2eb0cb57d"
+          (reference "Q4") (unit 1)
+        )
+      )
     )
   )
@@
     )
   )
-  (symbol (lib_id "Simulation_SPICE:NPN") (at 177.8 76.835 0) (unit 1)
+  (symbol (lib_id "PCM_Transistor_BJT_AKL:BC817") (at 177.8 76.835 0) (unit 1)
     (in_bom yes) (on_board yes) (dnp no) (fields_autoplaced)
-    (property "Reference" "Q1" (at 182.88 76.2 0)
+    (property "Reference" "Q1" (at 183.515 76.2 0)
       (effects (font (size 1.27 1.27)) (justify left))
     )
-    (property "Value" "s8050" (at 182.88 78.74 0)
+    (property "Value" "BC817" (at 183.515 78.74 0)
       (effects (font (size 1.27 1.27)) (justify left))
     )
-    (property "Footprint" "Package_TO_SOT_SMD:SOT-23" (at 241.3 76.835 0)
+    (property "Footprint" "Package_TO_SOT_SMD:SOT-23" (at 182.88 74.295 0)
       (effects (font (size 1.27 1.27)) hide)
     )
-    (property "Datasheet" "~" (at 241.3 76.835 0)
-      (effects (font (size 1.27 1.27)) hide)
-    )
-    (property "Sim.Device" "NPN" (at 177.8 76.835 0)
-      (effects (font (size 1.27 1.27)) hide)
-    )
-    (property "Sim.Type" "GUMMELPOON" (at 177.8 76.835 0)
-      (effects (font (size 1.27 1.27)) hide)
-    )
-    (property "Sim.Pins" "1=C 2=B 3=E" (at 177.8 76.835 0)
+    (property "Datasheet" "https://www.tme.eu/Document/7b5ea7386544f524d0315334956093bb/BC817-16.215.pdf" (at 177.8 76.835 0)
       (effects (font (size 1.27 1.27)) hide)
     )
@@
         )
       )
-    )
-  )
-  (symbol (lib_id "Simulation_SPICE:NPN") (at 233.68 77.47 0) (unit 1)
-    (in_bom yes) (on_board yes) (dnp no) (fields_autoplaced)
-    (property "Reference" "Q2" (at 238.76 76.835 0)
-      (effects (font (size 1.27 1.27)) (justify left))
-    )
-    (property "Value" "s8050" (at 238.76 79.375 0)
-      (effects (font (size 1.27 1.27)) (justify left))
-    )
-    (property "Footprint" "Package_TO_SOT_SMD:SOT-23" (at 297.18 77.47 0)
-      (effects (font (size 1.27 1.27)) hide)
-    )
-    (property "Datasheet" "~" (at 297.18 77.47 0)
-      (effects (font (size 1.27 1.27)) hide)
-    )
-    (property "Sim.Device" "NPN" (at 233.68 77.47 0)
-      (effects (font (size 1.27 1.27)) hide)
-    )
-    (property "Sim.Type" "GUMMELPOON" (at 233.68 77.47 0)
-      (effects (font (size 1.27 1.27)) hide)
-    )
-    (property "Sim.Pins" "1=C 2=B 3=E" (at 233.68 77.47 0)
-      (effects (font (size 1.27 1.27)) hide)
-    )
-    (pin "1")
-    (pin "2")
-    (pin "3")
-    (instances
-      (project "iot_diagnostic_tool"
-        (path "/2db85604-c96b-49da-91cc-aa2116c9cadf/7d43596b-0e17-496e-8cfa-ffe2eb0cb57d"
-          (reference "Q2") (unit 1)
-        )
-      )

Commit message: Update 26/06/23 - Thesis release
Other:
- company: VUT -> FEKT VUT
Changed lines of the file:
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@@
     (title "OBD Monitoring Device")
     (date "2023-02-27")
-    (company "VUT")
+    (company "FEKT VUT")
   )
   (junction (at 74.295 95.25) (diameter 0) (color 0 0 0 0)
