File: KiCAD project/Diagnostic tool with IoT/iot_diagnostic_tool/iot.kicad_sch (KiCad schematic)
At the start: 0 parts

Commit message: Update 03/03/23 - new schematic done
Parts:
- added C21: 10p, symbol Device:C
- added C22: 33p, symbol Device:C
- added C23, C26, C27, C30, C31: 100n, symbol Device:C
- added C24: 100u, symbol Device:C_Polarized
- added C25: 10n, symbol Device:C
- added D2: XBP1013G, symbol PCM_Diode_TVS_AKL:D_TVS_Unidirectional_Generic
- added D3, D4: LED, symbol Device:LED
- added D9: ESD9L3.3, Diode_SMD_AKL:D_SOD-923, symbol PCM_Diode_TVS_AKL:ESD9L3.3
- added Q3, Q4, Q5, Q7: s8050, symbol Simulation_SPICE:NPN
- added Q6: RUM001L02T2CL, symbol Device:Q_NMOS_GSD
- added R14, R22, R26: 4k7, symbol Device:R
- added R15, R23, R27: 47k, symbol Device:R
- added R16, R17: 51k, symbol Device:R
- added R18, R20: 120k, symbol Device:R
- added R19, R21, R40, R41, R44, R45: 10k, symbol Device:R
- added R24, R25: 2k2, symbol Device:R
- added R42, R43: 100k, symbol Device:R
- added SW3: IoT_RST, symbol Switch:SW_Push
- added U4: BG77LA-64-SGNS, MODULE_BG77LA-64-SGNS, symbol BG77LA-64-SGNS:BG77LA-64-SGNS
- added U5: NXS0108, Package_SO:TSSOP-20_4.4x6.5mm_P0.65mm, symbol tme_library:NXS0108PWJ
- added U7: NXS0104PWJ, Package_SO:TSSOP-14_4.4x5mm_P0.65mm, symbol tme_library:NXS0104
Connections:
- new net: Q3.2 (B), R14.2, R15.2
- new net: Q7.2 (B), R41.2, R42.1
- new net: Q6.1 (G), Q7.3 (E), R43.1
- new net: R20.2, R21.2, U7.8 (EN)
- new net: R18.2, R19.1, U5.10 (EN)
- new net: R17.1, U5.12 (B8), U5.13 (B7)
- new net: R16.1, U5.8 (A7), U5.9 (A8)
- new net: U4.29 (RSVD), U4.48 (RSVD), U4.49 (RSVD), U4.50 (RSVD), U4.51 (RSVD), U4.59 (RSVD), U4.67 (RSVD), U4.68 (RSVD), U4.69 (RSVD), U4.70 (RSVD), U4.71 (RSVD), U4.80 (RSVD), U4.81 (RSVD), U4.82 (RSVD), U4.91 (RSVD), U4.92 (RSVD), U4.93 (RSVD)
- new net: D4.1 (K), R25.1
- new net: Q7.1 (C), R40.2
- new net: Q4.1 (C), R24.2
- new net: Q4.2 (B), R22.2, R23.1
- new net: Q5.2 (B), R26.2, R27.1
- new net: D3.1 (K), R24.1
- new net: Q5.1 (C), R25.2
- new net +1V8: C27.1, C30.1, Q6.3 (D), R19.2, R21.1, R40.1, U5.2 (Vcc_A), U7.1 (VCC_A)
- new net +3V3: C21.1, C22.1, C23.1, C24.1, C26.1, C31.1, D2.1 (K), D3.2 (A), D4.2 (A), U4.19 (VBAT), U4.20 (VBAT), U5.19 (Vcc_B), U7.14 (VCC_B)
- new net ANT_GNSS: U4.32 (ANT_GNSS)
- new net ANT_MAIN: U4.26 (ANT_MAIN)
- new net AP_READY: R44.2, R45.1, U4.77 (AP_READY)
- new net AP_READY_MCU: R44.1
- new net DBG_RX: U7.11 (B3)
- new net DBG_RXD: U4.61 (DBG_RXD), U7.4 (A3)
- new net DBG_TX: U7.10 (B4)
- new net DBG_TXD: U4.60 (DBG_TXD), U7.5 (A4)
- new net GND: C21.2, C22.2, C23.2, C24.2, C25.2, C26.2, C27.2, C30.2, C31.2, D2.2 (A), D9.2 (A), Q3.3 (E), Q4.3 (E), Q5.3 (E), R15.1, R16.2, R17.2, R18.1, R20.1, R23.2, R27.2, R42.2, R43.2, R45.2, SW3.2, U4.22 (GND), U4.23 (GND), U4.24 (GND), U4.25 (GND), U4.27 (GND), U4.28 (GND), U4.30 (GND), U4.31 (GND), U4.43 (GND), U4.47 (GND), U4.52 (GND), U4.53 (GND), U4.54 (GND), U4.55 (GND), U4.56 (GND), U4.58 (GND), U4.66 (GND), U4.73 (GND), U4.74 (GND), U4.75 (GND), U4.84 (GND), U4.85 (GND), U4.86 (GND), U4.88 (GND), U4.89 (GND), U5.11 (GND), U7.7 (GND)
- new net GNSS_RX: U7.12 (B2)
- new net GNSS_RXD: U4.4 (GNSS_RXD), U7.3 (A2)
- new net GNSS_TX: U7.13 (B1)
- new net GNSS_TXD: U4.36 (GNSS_TXD), U7.2 (A1)
- new net IoT_CTS: U5.17 (B3)
- new net IoT_PWR: R14.1
- new net IoT_RI: U5.15 (B5)
- new net IoT_RTS: U5.16 (B4)
- new net IoT_RX: U5.20 (B1)
- new net IoT_TX: U5.18 (B2)
- new net MAIN_CTS: U4.39 (MAIN_CTS), U5.4 (A3)
- new net MAIN_DTR: U4.62 (MAIN_DTR), U5.7 (A6)
- new net MAIN_RI: U4.76 (MAIN_RI), U5.6 (A5)
- new net MAIN_RTS: U4.38 (MAIN_RTS), U5.5 (A4)
- new net MAIN_RXD: U4.6 (MAIN_RXD), U5.1 (A1)
- new net MAIN_TXD: U4.7 (MAIN_TXD), U5.3 (A2)
- new net NET_STATUS: R22.1, U4.79 (NET_STATUS)
- new net PON_TRIG: Q6.2 (S), U4.72 (PON_TRIG)
- new net PON_TRIG_MCU: R41.1
- new net PWRKEY: C25.1, Q3.1 (C), U4.46 (PWRKEY)
- new net RESET_N: D9.1 (K), SW3.1, U4.45 (RESET_N)
- new net SIM_CLK: U4.13 (USIM_CLK)
- new net SIM_DATA: U4.14 (USIM_DATA)
- new net SIM_DET: U4.44 (USIM_DET)
- new net SIM_GND: U4.65 (USIM_GND)
- new net SIM_RST: U4.15 (USIM_RST)
- new net SIM_VDD: U4.16 (USIM_VDD)
- new net STATUS: R26.1, U4.78 (STATUS)
- new net USBPHY: U4.42 (USBPHY_3P3)
- new net USB_BOOT: U4.87 (USB_BOOT)
- new net USB_D+: U4.11 (USB_DP)
- new net USB_D-: U4.10 (USB_DM)
- new net USB_VBUS: U4.12 (USB_VBUS)
- no-connect marks 0 -> 22
Other:
- added sheet antenna (ant.kicad_sch)
- added sheet sim (sim.kicad_sch)
- added sheet usb (usb.kicad_sch)
- note added: "AP READY"
- note added: "IoT Module Quectel BG77"
- note added: "Main module"
- note added: "PON Trigger"
- note added: "PWRKEY & RESET"
- note added: "Power"
- note added: "Status lights"
- note added: "UART Level Shifters"

Commit message: Update 06/03/23 - new board layout WIP 70%
Parts:
- removed C26, C30, C31: 100n, symbol Device:C
- removed D2: XBP1013G, symbol PCM_Diode_TVS_AKL:D_TVS_Unidirectional_Generic
- removed R17: 51k, symbol Device:R
- removed R18, R20: 120k, symbol Device:R
- removed R19, R21: 10k, symbol Device:R
- removed U5: NXS0108, Package_SO:TSSOP-20_4.4x6.5mm_P0.65mm, symbol tme_library:NXS0108PWJ
- removed U7: NXS0104PWJ, Package_SO:TSSOP-14_4.4x5mm_P0.65mm, symbol tme_library:NXS0104
- added D6: TPSMF4L5.0A, Diode_SMD:D_SOD-123F, symbol PCM_Diode_TVS_AKL:TPSMF4L5.0A
- added U8: NVT2010, Package_SO:TSSOP-24_4.4x7.8mm_P0.65mm, symbol tme_library:NVT2010
- C21, C22, C23, C25, C27: footprint (none) -> Capacitor_SMD:C_0402_1005Metric
- C24: footprint (none) -> Capacitor_Tantalum_SMD:CP_EIA-1608-08_AVX-J
- D3, D4: footprint (none) -> LED_SMD:LED_0402_1005Metric
- D9: footprint Diode_SMD_AKL:D_SOD-923 -> Diode_SMD:D_SOD-923
- Q3, Q4, Q5, Q7: footprint (none) -> Package_TO_SOT_SMD:SOT-23
- Q6: footprint (none) -> Package_TO_SOT_SMD:SOT-723
- R14, R15, R22, R23, R24, R25, R26, R27, R40, R41, R42, R43, R44, R45: footprint (none) -> Resistor_SMD:R_0402_1005Metric
- R16: value 51k -> 200k; footprint (none) -> Resistor_SMD:R_0402_1005Metric
- SW3: footprint (none) -> tme_library:XKB_TS_1187A
- U4: footprint MODULE_BG77LA-64-SGNS -> BG77LA-64-SGNS:MODULE_BG77LA-64-SGNS
Connections:
- net SIM_GND is gone; now on net GND: U4.65 (USIM_GND)
- net +1V8: now also U8.2 (VREFA); no longer C27.1
- net +3V3: now also R16.1, D6.1 (K)
- net DBG_RX: now also U8.16 (B7)
- net DBG_RXD: now also U8.9 (A7)
- net DBG_TX: now also U8.15 (B8)
- net DBG_TXD: now also U8.10 (A8)
- net GND: now also D6.2 (A), U8.1 (GND); no longer R16.2
- net GNSS_RX: now also U8.14 (B9)
- net GNSS_RXD: now also U8.11 (A9)
- net GNSS_TX: now also U8.13 (B10)
- net GNSS_TXD: now also U8.12 (A10)
- net IoT_CTS: now also U8.22 (B1)
- net IoT_DTR: now also U8.21 (B2)
- net IoT_RI: now also U8.17 (B6)
- net IoT_RTS: now also U8.19 (VREFB)
- net IoT_RX: now also U8.18 (B5)
- net IoT_TX: now also U8.20 (B3)
- net MAIN_CTS: now also U8.3 (A1)
- net MAIN_DTR: now also U8.4 (A2)
- net MAIN_RI: now also U8.8 (A6)
- net MAIN_RTS: now also U8.6 (A4)
- net MAIN_RXD: now also U8.7 (A5)
- net MAIN_TXD: now also U8.5 (A3)
- new net: C27.1, R16.2, U8.19 (VREFB), U8.24 (EN)
Other:
- note added: "UART Level Shifter"
- note removed: "UART Level Shifters"

Commit message: Update 07/03/23 - board layout done
Parts:
- removed D3, D4: LED, LED_SMD:LED_0402_1005Metric, symbol Device:LED
- removed Q4, Q5: s8050, Package_TO_SOT_SMD:SOT-23, symbol Simulation_SPICE:NPN
- removed R22, R26: 4k7, Resistor_SMD:R_0402_1005Metric, symbol Device:R
- removed R23, R27: 47k, Resistor_SMD:R_0402_1005Metric, symbol Device:R
- removed R24, R25: 2k2, Resistor_SMD:R_0402_1005Metric, symbol Device:R
Connections:
- net at C27.1, R16.2, U8.24 (EN): now also U8.23 (VREFB); no longer U8.19 (VREFB)
- net NET_STATUS: no longer names the net of U4.79 (NET_STATUS)
- net STATUS: no longer names the net of U4.78 (STATUS)
- no-connect marks 22 -> 24
Other:
- note removed: "Status lights"
- moved on the sheet: Q6, Q7, R40, R41, R42, R43, R44, R45

Commit message: Update 17/03/23 - final board update, generated files for manufacturing
Parts:
- removed Q3, Q7: s8050, Package_TO_SOT_SMD:SOT-23, symbol Simulation_SPICE:NPN
- added D2: LED, Diode_SMD:D_0603_1608Metric, symbol Device:LED
- added Q4 (x2): BC817, Package_TO_SOT_SMD:SOT-23_Handsoldering, symbol PCM_Transistor_BJT_AKL:BC817
- added Q4: BC817, Package_TO_SOT_SMD:SOT-23, symbol PCM_Transistor_BJT_AKL:BC817
- added R17: 2k2, Resistor_SMD:R_0402_1005Metric, symbol Device:R
- added R18: 4k7, Resistor_SMD:R_0402_1005Metric, symbol Device:R
- added R19: 47k, Resistor_SMD:R_0402_1005Metric, symbol Device:R
- C24: footprint Capacitor_Tantalum_SMD:CP_EIA-1608-08_AVX-J -> Capacitor_Tantalum_SMD:CP_EIA-3528-21_Kemet-B
- C27: footprint Capacitor_SMD:C_0402_1005Metric -> Capacitor_SMD:C_0402_1005Metric_Pad0.74x0.62mm_HandSolder
- R16, R40, R41, R42, R43, R44, R45: footprint Resistor_SMD:R_0402_1005Metric -> Resistor_SMD:R_0402_1005Metric_Pad0.72x0.64mm_HandSolder
Connections:
- net +3V3: now also D2.2 (A)
- net GND: now also Q4.2 (E), Q4.2 (E), R19.1
- net PWRKEY: now also Q4.3 (C)
- net at R14.2, R15.2: now also Q4.1 (B)
- net at R41.2, R42.1: now also Q4.1 (B)
- net at Q6.1 (G), R43.1: now also Q4.2 (E)
- net NET_STATUS: now reaches U4.79 (NET_STATUS)
- net NET_STATUS: now also R18.1
- net at R40.2: now also Q4.3 (C)
- new net: D2.1 (K), R17.1
- new net: Q4.3 (C), R17.2
- new net: Q4.1 (B), R18.2, R19.2
- no-connect marks 24 -> 23
Other:
- note added: "STATUS INDICATOR"

Commit message: Update 26/06/23 - Thesis release
Parts:
- added R20, R21, R22: 10k, symbol Device:R
Connections:
- net +3V3: now also R20.1, R21.1, R22.1
- net DBG_RX: now also U8.15 (B8), R21.2; no longer U8.16 (B7)
- net DBG_TX: now also U8.16 (B7); no longer U8.15 (B8)
- net GNSS_RX: now also U8.13 (B10), R22.2; no longer U8.14 (B9)
- net GNSS_TX: now also U8.14 (B9); no longer U8.13 (B10)
- net IoT_RX: now also U8.20 (B3), R20.2; no longer U8.18 (B5)
- net IoT_TX: now also U8.18 (B5); no longer U8.20 (B3)
Other:
- company: VUT -> FEKT VUT
- moved on the sheet: C27, R16, U8
