File: KiCAD project/Diagnostic tool with IoT/iot_diagnostic_tool/iot_diagnostic_tool.kicad_sch (KiCad schematic)
At the start: 15 parts, among them SW1 SW_Push, SW2 BOOT, U1 STM32L431RCTx, Y1 16 MHz

Commit message: Update 03/03/23 - new schematic done
Parts:
- removed SW2: BOOT, symbol Switch:SW_SPDT
- added J6: BOOT, symbol Connector:Conn_01x03_Pin
- SW1: value SW_Push -> RST
Connections:
- net GND: now also J6.3 (Pin_3)
- net IoT_RI: now also U1.20 (PA4); no longer U1.15 (PA1)
- net AP_READY_MCU: now reaches U1.10 (PC2)
- net PON_TRIG_MCU: now reaches U1.11 (PC3)
- net IoT_CTS: now reaches U1.14 (PA0)
- net IoT_PWR: now reaches U1.21 (PA5)
- net IoT_DTR: now reaches U1.22 (PA6)
- net GNSS_TX: now reaches U1.51 (PC10)
- net GNSS_RX: now reaches U1.52 (PC11)
- net at R1.2: now also J6.2 (Pin_2)
- net +3.3V renamed +3V3
- net +3V3: now also J6.1 (Pin_1)
- new net IoT_RTS: U1.15 (PA1)
- no-connect marks 36 -> 28
Other:
- note added: "MCU - STM32L431"
- note added: "Oscillator"
- note added: "Power"
- note added: "Reset & Boot0"
- moved on the sheet: C1, C10, C2, C3, C4, C5, C6, C7, C8, C9, R1, SW1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

Commit message: Update 06/03/23 - new board layout WIP 70%
Parts:
- C1: footprint (none) -> Capacitor_SMD:C_0603_1608Metric
- C10, C9: footprint (none) -> Capacitor_SMD:C_0402_1005Metric_Pad0.74x0.62mm_HandSolder
- C2, C3, C4, C5, C6, C7, C8: footprint (none) -> Capacitor_SMD:C_0402_1005Metric
- J6: footprint (none) -> Connector_PinHeader_2.54mm:PinHeader_1x03_P2.54mm_Vertical
- R1: footprint (none) -> Resistor_SMD:R_0402_1005Metric
- SW1: footprint (none) -> tme_library:XKB_TS_1187A
- Y1: footprint (none) -> Crystal:Crystal_SMD_3225-4Pin_3.2x2.5mm
Connections:
- net CAN_RX: now also U1.61 (PB8); no longer U1.44 (PA11)
- net CAN_S: now also U1.54 (PD2); no longer U1.39 (PC8)
- net CAN_TX: now also U1.62 (PB9); no longer U1.45 (PA12)
- net GND: now also Y1.2
- net K_Line_RX: now also U1.59 (PB7); no longer U1.43 (PA10)
- net K_Line_TX: now also U1.58 (PB6); no longer U1.42 (PA9)
- net L_Line: now also U1.45 (PA12); no longer U1.41 (PA8)
Other:
- moved on the sheet: SW1

Commit message: Update 07/03/23 - board layout done
Other:
- moved on the sheet: U1

Commit message: Update 26/06/23 - Thesis release
Other:
- company: VUT -> FEKT VUT
Changed lines of the file:
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@@
     (date "2023-02-27")
     (rev "1.0")
-    (company "VUT")
+    (company "FEKT VUT")
   )
   (junction (at 165.735 55.88) (diameter 0) (color 0 0 0 0)
