File: KiCAD project/Diagnostic tool with IoT/iot_diagnostic_tool/pwr.kicad_sch (KiCad schematic)
At the start: 12 parts, among them U2 TPS562201

Commit message: Update 03/03/23 - new schematic done
Parts:
- added C28, C29: 1u, symbol Device:C
- added U6: AP2120N-1.8, Package_TO_SOT_SMD:SOT-23, symbol Regulator_Linear:AP2127N-1.8
Connections:
- net +3.3V: now also C28.1, U6.3 (VI); no longer C15.1, C16.1, C17.1, L1.2, R2.1
- net GND: now also C28.2, C29.2, U6.1 (GND)
- new net +1V8: C29.1, U6.2 (VO)
- new net +3V3: C15.1, C16.1, C17.1, L1.2, R2.1
Other:
- note added: "1.8V Regulator"
- note added: "3.3V Regulator"
- note added: "Power supplies"
- note removed: "3.3V Power supply"
- moved on the sheet: C11, C12, C13, C14, C15, C16, C17, F1, L1, R2, R3, U2

Commit message: Update 06/03/23 - new board layout WIP 70%
Parts:
- C11, C14: footprint (none) -> Capacitor_SMD:C_0402_1005Metric
- C12, C13, C28, C29: footprint (none) -> Capacitor_SMD:C_0603_1608Metric
- C15, C16, C17: footprint (none) -> Capacitor_SMD:C_0805_2012Metric
- F1: footprint (none) -> Fuse:Fuse_0603_1608Metric_Pad1.05x0.95mm_HandSolder
- L1: footprint (none) -> tme_library:VLS6045AF
- R2, R3: footprint (none) -> Resistor_SMD:R_0402_1005Metric_Pad0.72x0.64mm_HandSolder
- U2: footprint (none) -> Package_TO_SOT_SMD:SOT-23-6
Connections:
- net +3.3V is gone; now on net +3V3: C28.1, U6.3 (VI)
- net SW: now reaches C14.1, L1.1, U2.2 (SW)
- net BST: now reaches C14.2, U2.6 (VBST)
- net FB: now reaches R2.2, R3.1, U2.4 (VFB)
Other:
- moved on the sheet: C14

Commit message: Update 17/03/23 - final board update, generated files for manufacturing
Parts:
- U6: footprint Package_TO_SOT_SMD:SOT-23 -> Package_TO_SOT_SMD:SOT-23_Handsoldering
Changed lines of the file:
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@@
       (effects (font (size 1.27 1.27)))
     )
-    (property "Footprint" "Package_TO_SOT_SMD:SOT-23" (at 100.33 104.775 0)
+    (property "Footprint" "Package_TO_SOT_SMD:SOT-23_Handsoldering" (at 100.33 104.775 0)
       (effects (font (size 1.27 1.27) italic) hide)
     )

Commit message: Update 26/06/23 - Thesis release
Other:
- company: VUT -> FEKT VUT
Changed lines of the file:
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@@
     (title "OBD Monitoring Device")
     (date "2023-02-27")
-    (company "VUT")
+    (company "FEKT VUT")
   )
   (junction (at 121.92 69.215) (diameter 0) (color 0 0 0 0)
