File: KiCAD project/Diagnostic tool with IoT/iot_diagnostic_tool/usb.kicad_sch (KiCad schematic)
At the start: 14 parts, among them J2 USB, J3 USB_BOOT, J4 USB_EN

Commit message: Update 06/03/23 - new board layout WIP 70%
Parts:
- removed J2: USB, symbol Connector:Conn_01x04_Pin
- removed J3: USB_BOOT, symbol Connector_Generic:Conn_01x02
- removed J4: USB_EN, symbol Connector_Generic:Conn_01x02
- C36, C37: footprint (none) -> Capacitor_SMD:C_0402_1005Metric
- D6: footprint Diode_SMD_AKL:D_SOD-123F -> Diode_SMD:D_SOD-123F
- D7: footprint Package_TO_SOT_SMD_AKL:SOT-23 -> Package_TO_SOT_SMD:SOT-23
- D8, D9: footprint Diode_SMD_AKL:D_SOD-923 -> Diode_SMD:D_SOD-923
- R33, R34, R35, R36, R37: footprint (none) -> Resistor_SMD:R_0402_1005Metric
Connections:
- net USB_D+: now also D7.2 (K2), R36.2
- net USB_D-: now also D7.1 (K1), R35.2
- net USB_VBUS_5: now reaches C36.2, D6.1 (K), R33.2
- net USB_BOOT_VCC: now reaches R37.1
Other:
- moved on the sheet: D9, R37

Commit message: Update 13/03/23 - Board layout fixes
Connections:
- net USB_D+: no longer D7.2 (K2), R36.2
- net USB_D-: no longer D7.1 (K1), R35.2
- new net USB_D+_5: D7.2 (K2), R36.2
- new net USB_D-_5: D7.1 (K1), R35.2
Other:
- moved on the sheet: C37, R33, R34
Changed lines of the file:
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@@
   (junction (at 140.335 90.805) (diameter 0) (color 0 0 0 0)
   )
-  (junction (at 90.805 90.805) (diameter 0) (color 0 0 0 0)
-  )
   (junction (at 130.175 93.345) (diameter 0) (color 0 0 0 0)
   )
+  (junction (at 99.06 90.805) (diameter 0) (color 0 0 0 0)
+  )
+  (junction (at 187.325 121.285) (diameter 0) (color 0 0 0 0)
+  )
+  (junction (at 187.325 80.645) (diameter 0) (color 0 0 0 0)
+  )
   (junction (at 94.615 90.805) (diameter 0) (color 0 0 0 0)
   )
-  (junction (at 187.325 121.285) (diameter 0) (color 0 0 0 0)
-  )
-  (junction (at 187.325 80.645) (diameter 0) (color 0 0 0 0)
-  )
   (junction (at 135.255 95.885) (diameter 0) (color 0 0 0 0)
   )
@@
     (stroke (width 0) (type dash))
   )
-  (wire (pts (xy 90.805 90.805) (xy 94.615 90.805))
+  (wire (pts (xy 88.9 90.805) (xy 94.615 90.805))
     (stroke (width 0) (type default))
   )
@@
     (stroke (width 0) (type default))
   )
-  (wire (pts (xy 104.775 90.805) (xy 111.76 90.805))
+  (wire (pts (xy 109.22 90.805) (xy 111.76 90.805))
     (stroke (width 0) (type default))
   )
@@
     (stroke (width 0) (type default))
   )
-  (wire (pts (xy 88.9 90.805) (xy 90.805 90.805))
-    (stroke (width 0) (type default))
-  )
   (wire (pts (xy 184.15 99.06) (xy 179.07 99.06))
     (stroke (width 0) (type default))
   )
+  (wire (pts (xy 94.615 90.805) (xy 99.06 90.805))
+    (stroke (width 0) (type default))
+  )
   (polyline (pts (xy 223.52 135.255) (xy 223.52 106.045))
     (stroke (width 0) (type dash))
   )
-  (wire (pts (xy 94.615 85.725) (xy 94.615 90.805))
+  (wire (pts (xy 99.06 85.725) (xy 99.06 90.805))
     (stroke (width 0) (type default))
   )
@@
     (stroke (width 0) (type default))
   )
-  (wire (pts (xy 94.615 90.805) (xy 97.155 90.805))
+  (wire (pts (xy 99.06 90.805) (xy 101.6 90.805))
     (stroke (width 0) (type default))
   )
@@
     (effects (font (size 1.27 1.27)) (justify left bottom))
   )
-  (label "USB_D+" (at 118.11 95.885 0) (fields_autoplaced)
+  (label "USB_DATA+" (at 118.11 95.885 0) (fields_autoplaced)
     (effects (font (size 1.27 1.27)) (justify left bottom))
   )
-  (label "USB_D-" (at 118.11 93.345 0) (fields_autoplaced)
+  (label "USB_DATA-" (at 118.11 93.345 0) (fields_autoplaced)
     (effects (font (size 1.27 1.27)) (justify left bottom))
   )
@@
     )
   )
-  (symbol (lib_id "power:GND") (at 90.805 98.425 0) (unit 1)
+  (symbol (lib_id "power:GND") (at 94.615 98.425 0) (unit 1)
     (in_bom yes) (on_board yes) (dnp no)
-    (property "Reference" "#PWR050" (at 90.805 104.775 0)
-      (effects (font (size 1.27 1.27)) hide)
-    )
-    (property "Value" "GND" (at 90.805 102.235 0)
-      (effects (font (size 1.27 1.27)))
-    )
-    (property "Footprint" "" (at 90.805 98.425 0)
-      (effects (font (size 1.27 1.27)) hide)
-    )
-    (property "Datasheet" "" (at 90.805 98.425 0)
+    (property "Reference" "#PWR050" (at 94.615 104.775 0)
+      (effects (font (size 1.27 1.27)) hide)
+    )
+    (property "Value" "GND" (at 94.615 102.235 0)
+      (effects (font (size 1.27 1.27)))
+    )
+    (property "Footprint" "" (at 94.615 98.425 0)
+      (effects (font (size 1.27 1.27)) hide)
+    )
+    (property "Datasheet" "" (at 94.615 98.425 0)
       (effects (font (size 1.27 1.27)) hide)
     )
@@
     )
   )
-  (symbol (lib_id "power:GND") (at 94.615 78.105 180) (unit 1)
-    (in_bom yes) (on_board yes) (dnp no) (fields_autoplaced)
-    (property "Reference" "#PWR047" (at 94.615 71.755 0)
-      (effects (font (size 1.27 1.27)) hide)
-    )
-    (property "Value" "GND" (at 94.615 74.295 0)
-      (effects (font (size 1.27 1.27)))
-    )
-    (property "Footprint" "" (at 94.615 78.105 0)
-      (effects (font (size 1.27 1.27)) hide)
-    )
-    (property "Datasheet" "" (at 94.615 78.105 0)
+  (symbol (lib_id "power:GND") (at 99.06 78.105 180) (unit 1)
+    (in_bom yes) (on_board yes) (dnp no) (fields_autoplaced)
+    (property "Reference" "#PWR047" (at 99.06 71.755 0)
+      (effects (font (size 1.27 1.27)) hide)
+    )
+    (property "Value" "GND" (at 99.06 74.295 0)
+      (effects (font (size 1.27 1.27)))
+    )
+    (property "Footprint" "" (at 99.06 78.105 0)
+      (effects (font (size 1.27 1.27)) hide)
+    )
+    (property "Datasheet" "" (at 99.06 78.105 0)
       (effects (font (size 1.27 1.27)) hide)
     )
@@
     )
   )
-  (symbol (lib_id "Device:C") (at 90.805 94.615 0) (unit 1)
-    (in_bom yes) (on_board yes) (dnp no) (fields_autoplaced)
-    (property "Reference" "C37" (at 94.615 93.98 0)
-      (effects (font (size 1.27 1.27)) (justify left))
-    )
-    (property "Value" "10n" (at 94.615 96.52 0)
-      (effects (font (size 1.27 1.27)) (justify left))
-    )
-    (property "Footprint" "Capacitor_SMD:C_0402_1005Metric" (at 91.7702 98.425 0)
-      (effects (font (size 1.27 1.27)) hide)
-    )
-    (property "Datasheet" "~" (at 90.805 94.615 0)
+  (symbol (lib_id "Device:C") (at 94.615 94.615 0) (unit 1)
+    (in_bom yes) (on_board yes) (dnp no) (fields_autoplaced)
+    (property "Reference" "C37" (at 98.425 93.98 0)
+      (effects (font (size 1.27 1.27)) (justify left))
+    )
+    (property "Value" "10n" (at 98.425 96.52 0)
+      (effects (font (size 1.27 1.27)) (justify left))
+    )
+    (property "Footprint" "Capacitor_SMD:C_0402_1005Metric" (at 95.5802 98.425 0)
+      (effects (font (size 1.27 1.27)) hide)
+    )
+    (property "Datasheet" "~" (at 94.615 94.615 0)
       (effects (font (size 1.27 1.27)) hide)
     )
@@
     )
   )
-  (symbol (lib_id "Device:R") (at 94.615 81.915 0) (unit 1)
-    (in_bom yes) (on_board yes) (dnp no) (fields_autoplaced)
-    (property "Reference" "R34" (at 97.155 81.28 0)
-      (effects (font (size 1.27 1.27)) (justify left))
-    )
-    (property "Value" "10k" (at 97.155 83.82 0)
-      (effects (font (size 1.27 1.27)) (justify left))
-    )
-    (property "Footprint" "Resistor_SMD:R_0402_1005Metric" (at 92.837 81.915 90)
-      (effects (font (size 1.27 1.27)) hide)
-    )
-    (property "Datasheet" "~" (at 94.615 81.915 0)
+  (symbol (lib_id "Device:R") (at 99.06 81.915 0) (unit 1)
+    (in_bom yes) (on_board yes) (dnp no) (fields_autoplaced)
+    (property "Reference" "R34" (at 101.6 81.28 0)
+      (effects (font (size 1.27 1.27)) (justify left))
+    )
+    (property "Value" "10k" (at 101.6 83.82 0)
+      (effects (font (size 1.27 1.27)) (justify left))
+    )
+    (property "Footprint" "Resistor_SMD:R_0402_1005Metric" (at 97.282 81.915 90)
+      (effects (font (size 1.27 1.27)) hide)
+    )
+    (property "Datasheet" "~" (at 99.06 81.915 0)
       (effects (font (size 1.27 1.27)) hide)
     )
@@
     )
   )
-  (symbol (lib_id "Device:R") (at 100.965 90.805 90) (unit 1)
-    (in_bom yes) (on_board yes) (dnp no) (fields_autoplaced)
-    (property "Reference" "R33" (at 100.965 86.36 90)
-      (effects (font (size 1.27 1.27)))
-    )
-    (property "Value" "20k" (at 100.965 88.9 90)
-      (effects (font (size 1.27 1.27)))
-    )
-    (property "Footprint" "Resistor_SMD:R_0402_1005Metric" (at 100.965 92.583 90)
-      (effects (font (size 1.27 1.27)) hide)
-    )
-    (property "Datasheet" "~" (at 100.965 90.805 0)
-      (effects (font (size 1.27 1.27)) hide)
-    )
+  (symbol (lib_id "Device:R") (at 105.41 90.805 90) (unit 1)
+    (in_bom yes) (on_board yes) (dnp no) (fields_autoplaced)
+    (property "Reference" "R33" (at 105.41 86.36 90)
+      (effects (font (size 1.27 1.27)))
+    )
+    (property "Value" "20k" (at 105.41 88.9 90)
+      (effects (font (size 1.27 1.27)))
+    )
+    (property "Footprint" "Resistor_SMD:R_0402_1005Metric" (at 105.41 92.583 90)
+      (effects (font (size 1.27 1.27)) hide)
+    )
+    (property "Datasheet" "~" (at 105.41 90.805 0)
+      (effects (font (size 1.27 1.27)) hide)
+    )

Commit message: Update 17/03/23 - final board update, generated files for manufacturing
Connections:
- net +1V8: now also R37.1; no longer R37.2
- net USB_BOOT_VCC: now also R37.2; no longer R37.1
Other:
- moved on the sheet: R37
Changed lines of the file:
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@@
     )
   )
-  (symbol (lib_id "Device:R") (at 175.26 99.06 270) (mirror x) (unit 1)
+  (symbol (lib_id "Device:R") (at 175.26 99.06 90) (mirror x) (unit 1)
     (in_bom yes) (on_board yes) (dnp no) (fields_autoplaced)
     (property "Reference" "R37" (at 175.26 93.98 90)
@@
       (effects (font (size 1.27 1.27)))
     )
-    (property "Footprint" "Resistor_SMD:R_0402_1005Metric" (at 175.26 100.838 90)
+    (property "Footprint" "Resistor_SMD:R_0402_1005Metric" (at 175.26 97.282 90)
       (effects (font (size 1.27 1.27)) hide)
     )

Commit message: Update 26/06/23 - Thesis release
Other:
- company: (none) -> FEKT VUT
- title: (none) -> OBD Monitoring Device
Changed lines of the file:
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@@
 (kicad_sch (version 20230121) (generator eeschema)
   (paper "A4")
+  (title_block
+    (title "OBD Monitoring Device")
+    (date "2023-02-27")
+    (company "FEKT VUT")
+  )
   (junction (at 140.335 90.805) (diameter 0) (color 0 0 0 0)
   )
